Commit message: modifications to actuators and main launch

File: ROS2 Software Stack/rrr_manipulator/description/rrr_manipulator_constants.xacro (robot description, xacro)
@@ -2,4 +2,13 @@
 <robot xmlns:xacro="http://www.ros.org/wiki/xacro" >
     <!-- Constant parameters -->
+    <xacro:property name="Ox" value="0.0" /> <!-- m -->
+    <xacro:property name="Oy" value="0.0" /> <!-- m -->
+    <xacro:property name="Oz" value="0.0" /> <!-- m -->
+    <xacro:property name="coxa_offset" value="0.35" /> <!-- m -->
+    <xacro:property name="coxa_reduction" value="-1.0" /> <!-- m -->
+    <xacro:property name="femur_offset" value="-0.3" /> <!-- m -->
+    <xacro:property name="femur_reduction" value="-1.0" /> <!-- m -->
+    <xacro:property name="tibia_offset" value="-0.55" /> <!-- m -->
+    <xacro:property name="tibia_reduction" value="1.0" /> <!-- m -->
     <xacro:property name="body_link_mass" value="2.0" /> <!-- Kg -->
     <xacro:property name="body_link_height" value="1.0" /> <!-- m -->
